Commit message: Fixed rotation of wheels for differential drive

File: urdf/garbagebot.urdf (robot description, URDF)
Before this commit: robot trashbot, 9 links, 8 joints
Links:
- removed link wheel_back_left_link
- removed link wheel_back_right_link
- removed link wheel_front_left_link
- removed link wheel_front_right_link
- added link caster_back_wheel, mass 0.1; collision sphere radius=0.018; visual sphere radius=0.018
- added link caster_front_wheel, mass 0.1; collision sphere radius=0.018; visual sphere radius=0.018
- added link wheel_left_link, mass 2.8498940e-02; collision cylinder length=0.018 radius=0.033; visual mesh filename=/home/qalis/ros2_ws/src/trashbot/meshes/trashbot_wheel_v5.s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 scale=0.0015 0.0015 0.0015
- added link wheel_right_link, mass 2.8498940e-02; collision cylinder length=0.018 radius=0.033; visual mesh filename=/home/qalis/ros2_ws/src/trashbot/meshes/trashbot_wheel_v5.s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 scale=0.0015 0.0015 0.0015
- link base_link: geometry collision box size=0.266 0.266 0.094; visual mesh filename=/home/qalis/ros2_ws/src/trashbot/meshes/trashbot_base v1.stl scale=0.0015 0.0015 0.0015
Joints:
- removed joint wheel_back_left_joint
- removed joint wheel_back_right_joint
- removed joint wheel_front_left_joint
- removed joint wheel_front_right_joint
- added joint caster_back_wheel_joint: type fixed, parent base_link, child caster_back_wheel, origin xyz=0 0.08 0.015, axis 0 0 1
- added joint caster_front_wheel_joint: type fixed, parent base_link, child caster_front_wheel, origin xyz=0 -0.08 0.015, axis 0 0 1
- added joint wheel_left_joint: type continuous, parent base_link, child wheel_left_link, origin xyz=0.16 0 0.045 rpy=0 0 0, axis 1 0 0
- added joint wheel_right_joint: type continuous, parent base_link, child wheel_right_link, origin xyz=-0.16 0 0.045 rpy=0 0 0, axis 1 0 0
- joint base_joint: origin xyz=0 0 0.010 rpy=0 0 0 -> xyz=0 0 0 rpy=0 0 0
- joint lidar_joint: origin xyz=0 0.02 0.1 rpy=0 0 0 -> xyz=0 0.02 0.12 rpy=0 0 0

File: urdf/garbagebot2.urdf (robot description, URDF)
Before this commit: robot trashbot, 9 links, 8 joints
Links:
- removed link wheel_back_left_link
- removed link wheel_back_right_link
- removed link wheel_front_left_link
- removed link wheel_front_right_link
- added link caster_back_wheel, mass 0.1; collision sphere radius=0.018; visual sphere radius=0.018
- added link caster_front_wheel, mass 0.1; collision sphere radius=0.018; visual sphere radius=0.018
- added link wheel_left_link, mass 2.8498940e-02; collision cylinder length=0.018 radius=0.033; visual mesh filename=package://trashbot/meshes/trashbot_wheel_v5.stl scale=0.0015 0.0015 0.0015
- added link wheel_right_link, mass 2.8498940e-02; collision cylinder length=0.018 radius=0.033; visual mesh filename=package://trashbot/meshes/trashbot_wheel_v5.stl scale=0.0015 0.0015 0.0015
- link base_link: geometry collision box size=0.266 0.266 0.094; visual mesh filename=package://trashbot/meshes/trashbot_base_v1.stl scale=0.0015 0.0015 0.0015
Joints:
- removed joint wheel_back_left_joint
- removed joint wheel_back_right_joint
- removed joint wheel_front_left_joint
- removed joint wheel_front_right_joint
- added joint caster_back_wheel_joint: type fixed, parent base_link, child caster_back_wheel, origin xyz=0 0.08 0.015, axis 0 0 1
- added joint caster_front_wheel_joint: type fixed, parent base_link, child caster_front_wheel, origin xyz=0 -0.08 0.015, axis 0 0 1
- added joint wheel_left_joint: type continuous, parent base_link, child wheel_left_link, origin xyz=0.16 0 0.045 rpy=0 0 0, axis 1 0 0
- added joint wheel_right_joint: type continuous, parent base_link, child wheel_right_link, origin xyz=-0.16 0 0.045 rpy=0 0 0, axis 1 0 0
- joint lidar_joint: origin xyz=0 0.02 0.1 rpy=0 0 0 -> xyz=0 0.02 0.12 rpy=0 0 0

Commit message: Made changes to fix differential drive
Proper inertial values, aligning of visual, collision, and inertial origins.

File: urdf/garbagebot.urdf (robot description, URDF)
Before this commit: robot trashbot, 9 links, 8 joints
Links:
- removed link camera
- removed link imu_link
- removed link lidar
- removed link wheel_back_left_link
- removed link wheel_back_right_link
- removed link wheel_front_left_link
- removed link wheel_front_right_link
- added link caster_back_wheel, mass 0.1; collision sphere radius=0.024; visual sphere radius=0.024
- added link caster_front_wheel, mass 0.1; collision sphere radius=0.024; visual sphere radius=0.024
- added link wheel_left_link, mass 0.4; collision cylinder length=0.018 radius=0.05; visual mesh filename=/home/qalis/ros2_ws/src/trashbot/meshes/trashbot_wheel_v5.s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 scale=0.0015 0.0015 0.0015
- added link wheel_right_link, mass 0.4; collision cylinder length=0.018 radius=0.05; visual mesh filename=/home/qalis/ros2_ws/src/trashbot/meshes/trashbot_wheel_v5.s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 scale=0.0015 0.0015 0.0015
- link base_link: mass 1.3729096e+00 -> 5; geometry collision box size=0.266 0.266 0.094; visual mesh filename=/home/qalis/ros2_ws/src/trashbot/meshes/trashbot_base v1.stl scale=0.0015 0.0015 0.0015
Joints:
- removed joint camera_joint
- removed joint imu_joint
- removed joint lidar_joint
- removed joint wheel_back_left_joint
- removed joint wheel_back_right_joint
- removed joint wheel_front_left_joint
- removed joint wheel_front_right_joint
- added joint caster_back_wheel_joint: type fixed, parent base_link, child caster_back_wheel, origin xyz=0 0.1 -0.058, axis 0 0 1
- added joint caster_front_wheel_joint: type fixed, parent base_link, child caster_front_wheel, origin xyz=0 -0.1 -0.058, axis 0 0 1
- added joint wheel_left_joint: type continuous, parent base_link, child wheel_left_link, origin xyz=0.14 0 -0.033 rpy=-1.5708 0 0, axis 1 0 0
- added joint wheel_right_joint: type continuous, parent base_link, child wheel_right_link, origin xyz=-0.14 0 -0.033 rpy=-1.5708 0 0, axis 1 0 0
- joint base_joint: origin xyz=0 0 0.010 rpy=0 0 0 -> xyz=0 0 0.05 rpy=0 0 0
